File: SPDIF_Input.sch (KiCad schematic (older format))
At the start: 8 parts, among them J201 SPDIF_IN, U201 TORX147

Commit message: Added board layout.
Parts:
- U201: footprint (none) -> fdsp_connector:TOxx147
Changed lines of the file:
@@
 F 0 "U201" H 3050 3800 60  0000 C CNN
 F 1 "TORX147" H 3050 3400 60  0000 C CNN
-F 2 "" H 3050 3450 60  0001 C CNN
+F 2 "fdsp_connector:TOxx147" H 3050 3450 60  0001 C CNN
 F 3 "" H 3050 3450 60  0000 C CNN
 	1    3050 3450
