File: SPDIF_Output.sch (KiCad schematic (older format))
At the start: 9 parts, among them J301 SPDIF_OUT, U301 TOTX147

Commit message: Added board layout.
Parts:
- U301: footprint (none) -> fdsp_connector:TOxx147
Changed lines of the file:
@@
 F 0 "U301" H 2950 3700 60  0000 C CNN
 F 1 "TOTX147" H 2950 3300 60  0000 C CNN
-F 2 "" H 2950 3350 60  0001 C CNN
+F 2 "fdsp_connector:TOxx147" H 2950 3350 60  0001 C CNN
 F 3 "" H 2950 3350 60  0000 C CNN
 	1    2950 3350
