File: Transceiver.sch (KiCad schematic (older format))
At the start: 34 parts, among them SW401 RESET, U401 74HC04, U402 WM8804, Y401 12MHz

Commit message: Added board layout.
Parts:
- JP401: value JUMPER3 -> TXSRC
- JP402: value JUMPER3 -> MASTER_SLAVE
- JP403: value JUMPER3 -> AIFCONF1
- JP404: value JUMPER3 -> HWMODE
- JP405: value JUMPER3 -> AIFCONF0
- R401: value R -> 10k
Changed lines of the file:
@@
 P 1600 1250
 F 0 "R401" V 1680 1250 50  0000 C CNN
-F 1 "R" V 1600 1250 50  0000 C CNN
+F 1 "10k" V 1600 1250 50  0000 C CNN
 F 2 "Resistors_SMD:R_0805_HandSoldering" V 1530 1250 30  0001 C CNN
 F 3 "" H 1600 1250 30  0000 C CNN
@@
 P 10300 2100
 F 0 "JP404" H 10350 2000 50  0000 L CNN
-F 1 "JUMPER3" H 10300 2200 50  0000 C BNN
+F 1 "HWMODE" H 10300 2200 50  0000 C BNN
 F 2 "Pin_Headers:Pin_Header_Straight_1x03" H 10300 2100 60  0001 C CNN
 F 3 "" H 10300 2100 60  0000 C CNN
@@
 P 9000 2100
 F 0 "JP402" H 9050 2000 50  0000 L CNN
-F 1 "JUMPER3" H 9000 2200 50  0000 C BNN
+F 1 "MASTER_SLAVE" H 9000 2200 50  0000 C BNN
 F 2 "Pin_Headers:Pin_Header_Straight_1x03" H 9000 2100 60  0001 C CNN
 F 3 "" H 9000 2100 60  0000 C CNN
@@
 P 9000 4400
 F 0 "JP403" H 9050 4300 50  0000 L CNN
-F 1 "JUMPER3" H 9000 4500 50  0000 C BNN
+F 1 "AIFCONF1" H 9000 4500 50  0000 C BNN
 F 2 "Pin_Headers:Pin_Header_Straight_1x03" H 9000 4400 60  0001 C CNN
 F 3 "" H 9000 4400 60  0000 C CNN
@@
 P 10300 4400
 F 0 "JP405" H 10350 4300 50  0000 L CNN
-F 1 "JUMPER3" H 10300 4500 50  0000 C BNN
+F 1 "AIFCONF0" H 10300 4500 50  0000 C BNN
 F 2 "Pin_Headers:Pin_Header_Straight_1x03" H 10300 4400 60  0001 C CNN
 F 3 "" H 10300 4400 60  0000 C CNN
@@
 P 7800 4400
 F 0 "JP401" H 7850 4300 50  0000 L CNN
-F 1 "JUMPER3" H 7800 4500 50  0000 C BNN
+F 1 "TXSRC" H 7800 4500 50  0000 C BNN
 F 2 "Pin_Headers:Pin_Header_Straight_1x03" H 7800 4400 60  0001 C CNN
 F 3 "" H 7800 4400 60  0000 C CNN
