File: SPDIF_Transceiver.kicad_pcb (KiCad board)
At the start: 2 copper layers, 50 x 80 mm, 96 parts, among them J201 SPDIF_IN, J301 SPDIF_OUT, P101 STDCONN, SW401 RESET, U101 LM2574, U201 TORX147, U301 TOTX147, U401 74HC04, U402 WM8804, Y401 12MHz

Commit message: Little changes, added Gerber Files.
Parts:
- added G***: LOGO, LOGO, B.Cu at (120.0, 110.0)
- added G***: LOGO, LOGO, F.Cu at (137.2, 142.2)
- added REF**: VIA_0503, fdsp_mechanical:VIA_0503, F.Cu at (113.0, 74.9)
- added REF**: VIA_0503, fdsp_mechanical:VIA_0503, F.Cu at (114.3, 74.9)
- added REF**: VIA_0503, fdsp_mechanical:VIA_0503, F.Cu at (114.3, 76.2)
- added REF**: VIA_0503, fdsp_mechanical:VIA_0503, F.Cu at (113.0, 76.2)
- moved R412 1.27 mm to (113.0, 79.4)
Connections:
- REF** pad 1: (no net) -> GND (x3)
Routing:
- net +3V3: track 192.6 -> 196.3 mm
- net /Transceiver/AIFCONF0: track 68.3 -> 65.4 mm
- net /Transceiver/SDA: track 96.4 -> 94.8 mm
- net Net-(JP404-Pad3): track 3.09 -> 4.12 mm
- added copper zone on F.Cu, net +12V
- added copper zone on F.Cu, net +3V3
- added copper zone on F.Cu, net Net-(D101-Pad1)
Other:
- board text added: "Fabian Geißler"
- board text added: "S/PDIF Transceiver V0.1"
